File: kicad/MainBoard/MainBoard.kicad_pcb (KiCad board)
At the start: 2 copper layers, 191.5 x 166.3 mm, 99 parts, among them J1 CHAN1, J10 ACC Port, J11 433TX, J12 VDC INPUT, J13 BAT, J14 TRG1, J15 TRG2, J16 FP-BUTTONS, J17 EXPAN2, J18 OUTPUT_BOARD_POWER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

Commit message: Fix connections of output jacks
Connections:
- J1 pad R: Net-(J4-Pin_1) -> unconnected-(J1-PadR)
- J2 pad R: Net-(J4-Pin_4) -> unconnected-(J2-PadR)
- J5 pad R: Net-(J4-Pin_11) -> unconnected-(J5-PadR)
- J7 pad R: Net-(J4-Pin_8) -> unconnected-(J7-PadR)
Routing:
- net Net-(J4-Pin_4): track 34.5 -> 22.0 mm
- net Net-(J4-Pin_8): track 31.1 -> 24.4 mm
- net Net-(J4-Pin_11): track 39.1 -> 32.5 mm
- net Net-(J4-Pin_1): track 25.9 -> 19.5 mm
Other:
- board text removed: "CHAN1"
